File: Boardtwo/Boardtwo.kicad_pcb (KiCad board)
At the start: 2 copper layers, 24.9 x 21.6 mm, 15 parts, among them J1 Conn_01x04_Pin, J2 Conn_01x04_Pin, J3 Conn_01x04_Pin, SW1 SW_Push, U1 AMS1117-3.3, U2 VL53L1CXV0FY1, U3 BMP280, U4 STM32F103C8Tx

Commit message: Update Boardtwo (altitude sensing PCB) layout and schematic
Parts:
- removed U2: VL53L1CXV0FY1, Sensor_Distance:ST_VL53L1x
- added J4: Conn_01x04_Pin, Connector_PinHeader_2.54mm:PinHeader_1x04_P2.54mm_Vertical, F.Cu at (110.2, 123.9)
- moved R2 2.65 mm to (127.7, 124.8)
Connections:
- U4 pad 18: /TOF_INT -> unconnected-(U4-PB0-Pad18)
- U4 pad 19: /TOF_XSHUT -> unconnected-(U4-PB1-Pad19)
Routing:
- net /ALT_SCL: track 28.3 -> 52.3 mm
- net /ALT_SDA: track 50.2 -> 27.5 mm, vias 3 -> 1
- net /TOF_XSHUT: track 14.9 -> 0.00 mm
- net /5V: track 18.6 -> 25.8 mm, vias 1 -> 0
- net /3V3: track 79.4 -> 73.4 mm
- net /SWDIO: track 22.2 -> 16.2 mm
- net Net-(U4-NRST): track 15.1 -> 20.7 mm, vias 2 -> 1
- net /TOF_INT: track 2.71 -> 0.00 mm
- net /GND: track 91.0 -> 92.9 mm
Other:
- board size 24.9 x 21.6 mm -> 28.2 x 21.6 mm
