File: Boardtwo/Boardtwo.kicad_sch (KiCad schematic)
At the start: 15 parts, among them J1 Conn_01x04_Pin, J2 Conn_01x04_Pin, J3 Conn_01x04_Pin, SW1 SW_Push, U1 AMS1117-3.3, U2 VL53L1CXV0FY1, U3 BMP280, U4 STM32F103C8Tx

Commit message: Update Boardtwo (altitude sensing PCB) layout and schematic
Parts:
- removed U2: VL53L1CXV0FY1, Sensor_Distance:ST_VL53L1x, symbol Sensor_Distance:VL53L1CXV0FY1
- added J4: Conn_01x04_Pin, Connector_PinHeader_2.54mm:PinHeader_1x04_P2.54mm_Vertical, symbol Connector:Conn_01x04_Pin
Connections:
- net 5V: now also J4.1 (Pin_1)
- net ALT_SCL: now also J4.4 (Pin_4)
- net ALT_SDA: now also J4.3 (Pin_3)
- net GND: now also J4.2 (Pin_2)
- net TOF_INT: no longer names the net of U4.18 (PB0)
- net TOF_XSHUT: no longer names the net of U4.19 (PB1)
- no-connect marks 36 -> 34
